File: bitaxeMax.kicad_pcb (KiCad board)
At the start: 4 copper layers, 56.5 x 99.8 mm, 153 parts, among them IC1 BM1397_mode1, J1 Conn_01x01, J10 FTSH-105-01-F-DV-K_SAI, J2 Conn_01x01, J3 Conn_01x05, J4 Conn_01x04, J5 TC2030-IDC, J6 Conn_01x08, J7 Conn_01x02, J9 Conn_01x04, Q1 CSD17311Q5, Q2 CSD17311Q5, U1 25MHz, U10 DS4432U+, U11 RT9080-33GJ5, U12 ESP32-S3-WROOM-1, U13 CLX6E-FKC, U2 TXB0104RGYR, U3 SN74AXC1T45DBVR, U4 CLX6E-FKC, U5 MCP1824, U6 MCP1824, U7 EMC2101, U8 INA260, U9 TPS40305, Y1 32.768kHz

Commit message: Add files via upload
Parts:
- removed C21, C26: 311-3342-1-ND, Capacitor_SMD:C_0402_1005Metric
- removed J10: FTSH-105-01-F-DV-K_SAI, bitaxe:FTSH-105-01-F-DV-K
- removed JP4: JTAG Source, Jumper:SolderJumper-3_P1.3mm_Bridged2Bar12_Pad1.0x1.5mm
- removed R18, R19: 1k, Resistor_SMD:R_0402_1005Metric
- removed R23: 0, Resistor_SMD:R_0402_1005Metric
- removed TP21: TestPoint, TestPoint:TestPoint_Pad_D1.5mm
- removed U3: SN74AXC1T45DBVR, bitaxe:SN74AXC1T45
- added ?: , , F.Cu at (81.3, 55.9)
- added ?: , , F.Cu at (81.3, 58.4)
- added D1: SS310, bitaxe:SMA_L4.3-W2.6-LS5.2-RD, F.Cu at (124.5, 96.5)
- added J11: 20021121-00006C1LF, bitaxe:2002112100006C1LF, B.Cu at (128.3, 89.5)
- added SW1: GT-TC029B-H025-L1N, bitaxe:SW_CS1213AGF260_CRS, B.Cu at (129.9, 116.8)
- added SW2: GT-TC029B-H025-L1N, bitaxe:SW_CS1213AGF260_CRS, B.Cu at (129.9, 124.5)
- added USB1: 10118193-0001LF, bitaxe:USB_10118193-0001LF_AMP, B.Cu at (131.7, 102.4)
- C1, C19, C20, C22, C23, C29, C33, C7, C9: value 311-3342-1-ND -> 0.1uF
- C10, C11, C12, C14, C15, C16, C17, C18, C2, C3, C4, C5, C6, C8: value 587-5514-1-ND -> 1uF
- H1, H2, H3, H4: footprint MountingHole:MountingHole_2.2mm_M2 -> MountingHole:MountingHole_2.2mm_M2_Pad_Via
- U5: value MCP1824 -> MCP1824T-1802E
- U6: value MCP1824 -> MCP1824T-0802E
- moved R20 33.8 mm to (130.1, 111.8)
- moved C50 32.8 mm to (127.0, 111.8), turned to 180 degrees
- moved TP31 21.4 mm to (129.5, 109.2)
- moved C19 7.83 mm to (116.4, 102.7)
- moved C20 7.83 mm to (114.0, 96.9)
- moved U2 7.83 mm to (116.3, 99.8)
- moved TP24 7.57 mm to (110.4, 102.0)
Connections:
- U12 pad 13: /BM1397/CLKI -> Net-(U12-GPIO19/U1RTS/ADC2_CH8/CLK_OUT2/USB_D-)
- U12 pad 14: unconnected-(U12-Pad14) -> Net-(U12-GPIO20/U1CTS/ADC2_CH9/CLK_OUT1/USB_D+)
- U12 pad 15: Net-(U12-Pad15) -> /3V3
- U12 pad 32: /ESP32/MTCK -> unconnected-(U12-MTCK/GPIO39/CLK_OUT3/SUBSPICS1-Pad32)
- U12 pad 33: /ESP32/MTDO -> unconnected-(U12-MTDO/GPIO40/CLK_OUT2-Pad33)
- U12 pad 34: /ESP32/MTDI -> unconnected-(U12-MTDI/GPIO41/CLK_OUT1-Pad34)
- U12 pad 35: /ESP32/MTMS -> unconnected-(U12-MTMS/GPIO42-Pad35)
Routing:
- net /ESP32/IO0: track 27.9 -> 114.3 mm, vias 2 -> 4
- net /ESP32/EN: track 34.1 -> 79.9 mm, vias 2 -> 3
- net /5V: track 180.2 -> 221.8 mm, vias 6 -> 7
- net /ESP32/P_TX: track 7.79 -> 45.4 mm, vias 1 -> 2
- net /ESP32/P_RX: track 9.97 -> 44.5 mm, vias 1 -> 2
- net Net-(R23-Pad2): track 33.4 -> 0.00 mm, vias 2 -> 0
- net Net-(U12-GPIO19/U1RTS/ADC2_CH8/CLK_OUT2/USB_D-): track 0.00 -> 33.2 mm
- net /ESP32/MTDO: track 33.2 -> 0.00 mm, vias 2 -> 0
- net Net-(U12-GPIO20/U1CTS/ADC2_CH9/CLK_OUT1/USB_D+): track 0.00 -> 32.5 mm
- net /ESP32/MTDI: track 32.3 -> 0.00 mm, vias 2 -> 0
- net /BM1397/CLKI: track 32.1 -> 0.00 mm, vias 1 -> 0
- net /ESP32/MTCK: track 31.8 -> 0.00 mm, vias 2 -> 0
- net /ESP32/MTMS: track 28.9 -> 0.00 mm, vias 2 -> 0
- net GND: track 133.4 -> 152.8 mm, vias 73 -> 72
- net /Power/VIN: track 6.26 -> 21.5 mm
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Other:
- board text added: "VCC"
