File: esp32.kicad_sch (KiCad schematic)
At the start: 39 parts, among them J10 FTSH-105-01-F-DV-K, J5 TC2030-IDC, J6 Conn_01x08, J9 Conn_01x04, U11 RT9080-33GJ5, U12 ESP32-S3-WROOM-1, U13 CLX6E-FKC, U4 CLX6E-FKC, Y1 32.768kHz

Commit message: Add files via upload
Parts:
- removed J10: FTSH-105-01-F-DV-K, bitaxe:FTSH-105-01-F-DV-K, symbol bitaxe:FTSH-105-01-F-DV-K
- removed JP4: JTAG Source, Jumper:SolderJumper-3_P1.3mm_Bridged2Bar12_Pad1.0x1.5mm, symbol Jumper:SolderJumper_3_Bridged12
- removed R18, R19: 1k, Resistor_SMD:R_0402_1005Metric, symbol Device:R_US
- removed TP21: TestPoint, TestPoint:TestPoint_Pad_D1.5mm, symbol Connector:TestPoint
- added D1: SS310, bitaxe:SMA_L4.3-W2.6-LS5.2-RD, symbol lcsc:SS310_C85658
- added J11: 20021121-00006C1LF, 2002112100006C1LF, symbol bitaxe:20021121-00006C1LF
- added SW1, SW2: GT-TC029B-H025-L1N, bitaxe:SW_CS1213AGF260_CRS, symbol lcsc:GT-TC029B-H025-L1N
- added USB1: 10118193-0001LF, bitaxe:USB_10118193-0001LF_AMP, symbol lcsc:U254-051T-4BHJ25-F2S
Connections:
- net 3V3: now also U12.15 (GPIO3/TOUCH3/ADC1_CH2*), J11.2
- net 5V: now also D1.1
- net EN: now also J11.1, SW1.2
- net GND: now also J11.4, SW1.1, SW2.1, USB1.5 (GND), USB1.6, USB1.7, USB1.8, USB1.9
- net IO0: now also J11.6, SW2.2
- net P_RX: now also J11.5
- net P_TX: now also J11.3
- net at U12.14 (GPIO20/U1CTS/ADC2_CH9/CLK_OUT1/USB_D+): now also USB1.3 (D+)
- net CLKI: no longer names the net of U12.13 (GPIO19/U1RTS/ADC2_CH8/CLK_OUT2/USB_D-)
- net CLKI: now also USB1.2 (D-)
- net MTCK: no longer names the net of U12.32 (MTCK/GPIO39/CLK_OUT3/SUBSPICS1)
- net MTDI: no longer names the net of U12.34 (MTDI/GPIO41/CLK_OUT1)
- net MTDO: no longer names the net of U12.33 (MTDO/GPIO40/CLK_OUT2)
- net MTMS: no longer names the net of U12.35 (MTMS/GPIO42)
- new net: D1.2, USB1.1 (VBUS)
Other:
- note added: "Program the ESP32 with a ESP-PROG and UART Interface connector 6 pins"
- note added: "USB port for programming the ESP32"
- note added: "micro B USB 2.0"
- note removed: "JTAG Pins"
- note removed: "Optional JTAG Programming Pins"
- note removed: "The ESP32 has built in I2C pull-ups"
- note removed: "USB/Serial"
- moved on the sheet: J9
